File: Hardware/wearableHardware/MCU.kicad_sch (KiCad schematic)
At the start: 1 part, among them U1 ESP32-S3-MINI-1

Commit message: feat: add MCU passives, pull-ups, decoupling, and support circuitry
Add all remaining components to the ESP32-S3-MINI-1 schematic sheet:
- VDD3P3 decoupling (100nF + 10µF)
- EN RC circuit (10kΩ pull-up, 1µF delay cap, reset switch)
- IO0 boot circuit (10kΩ pull-up, boot switch)
- I2C pull-ups (4.7kΩ on SDA/SCL)
- Display backlight driver (BSS138 N-FET, 1kΩ gate R, 15Ω drain R)
- Battery voltage divider (100k/100k with 100nF bypass)
- Event button (to GND with internal pull-up)
- Haptic driver (MMBT2222A NPN, 1kΩ base R, 1N4148W flyback)
- USB series termination (22Ω on D+/D-)
- UART test points (TXD0, RXD0)
- 3.3V power rail and GND distribution

All wire routing uses actual KiCad 9 library pin coordinates.

Co-Authored-By: Claude Opus 4.7 <noreply@anthropic.com>
Parts:
- added C1, C4: 100nF, Capacitor_SMD:C_0402_1005Metric, symbol Device:C
- added C2: 10uF, Capacitor_SMD:C_0603_1608Metric, symbol Device:C
- added C3: 1uF, Capacitor_SMD:C_0402_1005Metric, symbol Device:C
- added D1: 1N4148W, Diode_SMD:D_SOD-123, symbol Diode:1N4148W
- added Q1: BSS138, Package_TO_SOT_SMD:SOT-23, symbol Transistor_FET:BSS138
- added Q2: MMBT2222A, Package_TO_SOT_SMD:SOT-23, symbol Transistor_BJT:MMBT2222A
- added R1, R2: 10k, Resistor_SMD:R_0402_1005Metric, symbol Device:R
- added R10, R11: 22, Resistor_SMD:R_0402_1005Metric, symbol Device:R
- added R3, R4: 4.7k, Resistor_SMD:R_0402_1005Metric, symbol Device:R
- added R5, R9: 1k, Resistor_SMD:R_0402_1005Metric, symbol Device:R
- added R6: 15, Resistor_SMD:R_0402_1005Metric, symbol Device:R
- added R7, R8: 100k, Resistor_SMD:R_0402_1005Metric, symbol Device:R
- added SW1, SW2, SW3: SW_Push, Button_Switch_SMD:SW_SPST_SKQG_WithStem, symbol Switch:SW_Push
- added TP1, TP2, TP3, TP4: TestPoint, TestPoint:TestPoint_Pad_D1.0mm, symbol Connector_Generic:Conn_01x01
