File: Hardware/wearableHardware/display.kicad_sch (KiCad schematic)
At the start: 0 parts

Commit message: feat: add hardware schematics, documentation images, and external component libraries for wearable device development
Parts:
- added J2: ZF5S-15-01-T-WT, ZF5S-15-01-T-WT:SAMTEC_ZF5S-15-01-T-WT, symbol ZF5S-15-01-T-WT:ZF5S-15-01-T-WT
- added Q1: BSS138, Package_TO_SOT_SMD:SOT-23, symbol Transistor_FET:BSS138
- added R7: 1K, symbol Device:R
- added R8: 15, symbol Device:R
Connections:
- new net: J2.02, Q1.3 (D)
- new net: J2.03, R8.1
- new net: Q1.1 (G), R7.2
- new net +3.3V: J2.04, J2.10, R8.2
- new net BLK: R7.1
- new net CS: J2.06
- new net GND: J2.01, J2.11, Q1.2 (S)
- new net RS: J2.05
- new net RST: J2.09
- new net SCL: J2.07
- new net SDA: J2.08
- new net TP_INT: J2.13
- new net TP_RST: J2.12
- new net TP_SCL: J2.15
- new net TP_SDA: J2.14
